File: Emergency_Board-2023.8ver/emergency.brd (EAGLE design)
At the start: 67.5 x 88.5 mm, 32 parts, among them J1 8P8C, J2 XT60PW-F, J3 XT60PW-F, J4 XT60PW-F, J5 XT60PW-F, J6 MA02-2, J7 XT90PW-M, Q1 BUZ11BH, U10 MC34063AD, U4 TLP184

Commit message: update
Parts:
- removed C21, C5, C7: 100n, rcl:C0603
- removed C22: 47u, rcl:E2,5-5
- removed C6: 100p, rcl:C0603
- removed D3: PMEG6010CEJ,115, nexperia:SOD323_ST
- removed J1: 8P8C, con-rj45:8P8C
- removed L1: L5852, inductors:L5852
- removed R11: 0.68, rcl:R1206
- removed R18: 3.6k, rcl:R0603
- removed R19: 1.2k, rcl:R0603
- removed S1, S2: 897-1AH-C-001, relay:897-1AH-C-001
- removed U10: MC34063AD, mc34063:SOIC8
- added C1: 100n, rcl:C0603
- added C2: 47u, rcl:E2,5-5
- added J8: 8P8C-LED, con-rj45:8P8C-LED
- added R10: 470, rcl:R0603
- added R9: 1k, rcl:R0603
- added U$1, U$2: 897-1AH-C-001, CRS_EAGLE_Lib:897-1AH-C-001
- moved F1 45.1 mm to (3.50, 51.5), turned to 0 degrees
- moved J6 22.4 mm to (30.0, 79.0), turned to 0 degrees
- moved R12 20.5 mm to (27.5, 75.5)
- moved U4 16.8 mm to (4.78, 64.0), turned to 270 degrees
- moved R30 16.1 mm to (9.80, 60.9)
- moved R2 12.0 mm to (9.80, 58.7), turned to 0 degrees
- moved Q1 9.88 mm to (17.3, 66.3), turned to 0 degrees
- moved R28 9.82 mm to (24.5, 67.0), turned to 0 degrees
- moved R3 8.28 mm to (12.5, 58.5), turned to 270 degrees
Connections:
- removed net +5V: C21.2, C22.+, C5.1, L1.P$2, R18.2, U4.4
- removed net N$1: R11.2, U10.1, U10.7, U10.8
- removed net N$26: D3.C, L1.P$1, U10.2
- removed net N$27: C6.1, U10.3
- removed net N$28: R18.1, R19.2, U10.5
- removed net N$8: F1.2, J1.4, J1.5
- new net CAN_LED: J8.YA
- new net N$10: J8.YC, R10.2
- new net N$5: J8.GC, R9.2
- new net POWER: C1.1, C2.+, F1.2, U4.4
- net !EMS_ISO: now also J8.6; no longer J1.6
- net +12V: now also J8.4, J8.5, J8.GA; no longer C7.1, F1.1, R11.1, S1.P$2, S2.P$2, U10.6
- net BATT_POWER: now also F1.1, U$1.86_B, U$1.86_T, U$1.P$4, U$2.86_B, U$2.86_T, U$2.P$4
- net CANH: now also J8.1; no longer J1.1
- net CANL: now also J8.2; no longer J1.2
- net GND1: now also C1.2, C2.-, Q1.S, R3.2, R30.1, U$1.30_B, U$1.30_T, U$1.P$3, U$2.30_B, U$2.30_T, U$2.P$3; no longer S1.P$1, S2.P$1
- net GND2: now also U$1.87_B, U$1.87_T, U$1.P$1; no longer S1.P$4
- net GND3: now also U$2.87_B, U$2.87_T, U$2.P$1; no longer S2.P$4
- net GNDIO: now also J8.3, J8.7, J8.8, J8.M1, J8.M2, R10.1, R9.1; no longer C21.1, C22.-, C5.2, C6.2, C7.2, D3.A, J1.3, J1.7, J1.8, J1.M1, J1.M2, Q1.S, R19.1, R3.2, R30.1, U10.4
- net N$3: now also U$1.85_B, U$1.85_T, U$1.P$2, U$2.85_B, U$2.85_T, U$2.P$2; no longer S1.P$3, S2.P$3
Routing:
- net +12V: track 98.5 -> 8.70 mm
- net +5V: track 20.7 -> 0.00 mm
- net N$8: track 16.3 -> 0.00 mm
- net !EMS_ISO: track 10.3 -> 24.9 mm
- net N$30: track 3.22 -> 17.7 mm
- net BATT_POWER: track 0.00 -> 13.7 mm
- net N$28: track 13.1 -> 0.00 mm
- net N$3: track 52.4 -> 65.1 mm
- net POWER: track 0.00 -> 12.1 mm
- net N$1: track 9.68 -> 0.00 mm
- net N$7: track 12.8 -> 4.72 mm
- net N$26: track 6.71 -> 0.00 mm
- net !EMS: track 5.84 -> 9.40 mm
- net CANH: track 10.00 -> 13.4 mm
- net N$10: track 0.00 -> 3.23 mm
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- removed copper zone on layer 16, net GND2
Other:
- board text added: "Oct,11,2023"
- board text added: "by ykc"
- board text removed: "Nov,5,2019"
- board text removed: "by khk"

Commit message: update
Parts:
- removed C2: 47u, rcl:E2,5-5
- moved F1 39.0 mm to (37.5, 70.5), turned to 180 degrees
- moved U4 31.2 mm to (35.8, 67.2), turned to 180 degrees
- moved C1 28.2 mm to (33.0, 70.5), turned to 180 degrees
- moved R30 21.1 mm to (29.2, 69.2), turned to 90 degrees
- moved R28 19.2 mm to (43.1, 71.7)
- moved R2 19.1 mm to (25.3, 69.8), turned to 180 degrees
- moved R3 14.6 mm to (22.6, 69.0)
- moved Q1 6.71 mm to (15.8, 72.8)
- moved R9 3.26 mm to (32.8, 73.9)
- moved R10 2.00 mm to (48.5, 71.5), turned to 180 degrees
Connections:
- net +12V: now also F1.1, U$1.86_B, U$1.86_T, U$1.P$4, U$2.86_B, U$2.86_T, U$2.P$4
- net BATT_POWER: no longer F1.1, U$1.86_B, U$1.86_T, U$1.P$4, U$2.86_B, U$2.86_T, U$2.P$4
- net GND1: no longer C1.2, C2.-, Q1.S, R3.2, R30.1
- net GNDIO: now also C1.2, Q1.S, R3.2, R30.1
- net POWER: no longer C2.+
Routing:
- net +12V: track 8.70 -> 170.3 mm
- net !EMS_ISO: track 24.9 -> 8.00 mm
- net BATT_POWER: track 13.7 -> 0.00 mm
- net N$30: track 17.7 -> 7.05 mm
- net N$7: track 4.72 -> 12.9 mm
- net POWER: track 12.1 -> 7.69 mm
- net !EMS: track 9.40 -> 7.30 mm
- net N$3: track 65.1 -> 66.4 mm
- net N$5: track 3.19 -> 2.61 mm
