File: Emergency_Board-2023.8ver/emergency.sch (EAGLE design)
At the start: 32 parts, among them J1 8P8C, J2 XT60PW-F, J3 XT60PW-F, J4 XT60PW-F, J5 XT60PW-F, J6 MA02-2, J7 XT90PW-M, Q1 BUZ11BH, U10 MC34063AD, U4 TLP184

Commit message: update
Parts:
- removed C21, C5, C7: 100n, rcl:C-EUC0603
- removed C22: 47u, rcl:CPOL-EUE2.5-5
- removed C6: 100p, rcl:C-EUC0603
- removed D3: PMEG6010CEJ,115, nexperia:PMEG6010CEJ,115
- removed J1: 8P8C, con-rj45:8P8C
- removed L1: L5852, inductors:L5852
- removed R11: 0.68, rcl:R-EU_R1206
- removed R18: 3.6k, rcl:R-EU_R0603
- removed R19: 1.2k, rcl:R-EU_R0603
- removed S1, S2: 897-1AH-C-001, relay:897-1AH-C-001
- removed U10: MC34063AD, mc34063:MC34063AD
- added C1: 100n, rcl:C-EUC0603
- added C2: 47u, rcl:CPOL-EUE2.5-5
- added J8: 8P8C-LED, con-rj45:8P8C-LED
- added R10: 470, rcl:R-EU_R0603
- added R9: 1k, rcl:R-EU_R0603
- added U$1, U$2: 897-1AH-C-001, CRS_EAGLE_Lib:897-1AH-C-001
Connections:
- removed net +5V: C21.2, C22.+, C5.1, L1.2, R18.2, U4.C
- removed net N$1: R11.2, U10.DC, U10.IS, U10.SWC
- removed net N$26: D3.C, L1.1, U10.SWE
- removed net N$27: C6.1, U10.TC
- removed net N$28: R18.1, R19.2, U10.FB
- removed net N$8: F1.2, J1.4, J1.5
- new net CAN_LED: J8.A-Y
- new net N$10: J8.C-Y, R10.2
- new net N$5: J8.C-G, R9.2
- new net POWER: C1.1, C2.+, F1.2, U4.C
- net !EMS_ISO: now also J8.6; no longer J1.6
- net +12V: now also J8.4, J8.5, J8.A-G; no longer C7.1, F1.1, R11.1, S1U1.1, S2U1.1, U10.VCC
- net BATT_POWER: now also F1.1, U$1G$1.1, U$2G$1.1
- net CANH: now also J8.1; no longer J1.1
- net CANL: now also J8.2; no longer J1.2
- net GND1: now also C1.2, C2.-, Q1.S, R3.2, R30.1, U$1G$2.O, U$2G$2.O; no longer S1U2.S, S2U2.S
- net GND2: now also U$1G$2.P; no longer S1U2.P
- net GND3: now also U$2G$2.P; no longer S2U2.P
- net GNDIO: now also J8.3, J8.7, J8.8, J8.SHIELD, R10.1, R9.1; no longer C21.1, C22.-, C5.2, C6.2, C7.2, D3.A, J1.3, J1.7, J1.8, J1.SHIELD1, J1.SHIELD2, Q1.S, R19.1, R3.2, R30.1, U10.GND
- net N$3: now also U$1G$1.2, U$2G$1.2; no longer S1U1.2, S2U1.2

Commit message: update
Parts:
- removed C2: 47u, rcl:CPOL-EUE2.5-5
Connections:
- net +12V: now also F1.1, U$1G$1.1, U$2G$1.1
- net BATT_POWER: no longer F1.1, U$1G$1.1, U$2G$1.1
- net GND1: no longer C1.2, C2.-, Q1.S, R3.2, R30.1
- net GNDIO: now also C1.2, Q1.S, R3.2, R30.1
- net POWER: no longer C2.+
Other:
- moved on the sheet: C1, F1
Changed lines of the file:
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@@
 <part name="R10" library="rcl" library_urn="urn:adsk.eagle:library:334" deviceset="R-EU_" device="R0603" package3d_urn="urn:adsk.eagle:package:23555/3" value="470"/>
 <part name="C1" library="rcl" library_urn="urn:adsk.eagle:library:334" deviceset="C-EU" device="C0603" package3d_urn="urn:adsk.eagle:package:23616/2" value="100n"/>
-<part name="C2" library="rcl" library_urn="urn:adsk.eagle:library:334" deviceset="CPOL-EU" device="E2.5-5" package3d_urn="urn:adsk.eagle:package:23344/1" value="47u"/>
 <part name="GND1" library="supply1" library_urn="urn:adsk.eagle:library:371" deviceset="GNDIO" device=""/>
 <part name="U$1" library="CRS_EAGLE_Lib" library_urn="urn:adsk.wipprod:fs.file:vf.4_7vYAeHRqGNphZlrW9Mng" deviceset="897-1AH-C-001" device=""/>
@@
 <pinref part="J5" gate="G$1" pin="GND"/>
 </segment>
+</net>
+<net name="!EMS" class="2">
+<segment>
+<pinref part="R2" gate="G$1" pin="1"/>
+<wire x1="45.72" y1="68.58" x2="33.02" y2="68.58" width="0.1524" layer="91"/>
+<label x="38.1" y="68.58" size="1.778" layer="95"/>
+</segment>
+</net>
+<net name="GND1" class="2">
+<segment>
+<pinref part="J7" gate="G$1" pin="2"/>
+<pinref part="SUPPLY7" gate="G$1" pin="GND2"/>
+<wire x1="27.94" y1="88.9" x2="33.02" y2="88.9" width="0.1524" layer="91"/>
+<label x="33.02" y="88.9" size="1.778" layer="95"/>
+</segment>
+<segment>
+<label x="99.06" y="116.84" size="1.778" layer="95"/>
+<wire x1="99.06" y1="96.52" x2="99.06" y2="101.6" width="0.1524" layer="91"/>
+<wire x1="99.06" y1="101.6" x2="99.06" y2="114.3" width="0.1524" layer="91"/>
+<wire x1="109.22" y1="96.52" x2="109.22" y2="101.6" width="0.1524" layer="91"/>
+<wire x1="109.22" y1="101.6" x2="99.06" y2="101.6" width="0.1524" layer="91"/>
+<junction x="99.06" y="101.6"/>
+<pinref part="U$1" gate="G$2" pin="O"/>
+<pinref part="U$2" gate="G$2" pin="O"/>
+</segment>
+</net>
+<net name="GND3" class="2">
+<segment>
+<pinref part="J4" gate="G$1" pin="1"/>
+<pinref part="SUPPLY3" gate="G$1" pin="GND2"/>
+<wire x1="157.48" y1="40.64" x2="152.4" y2="40.64" width="0.1524" layer="91"/>
+<label x="147.32" y="43.18" size="1.778" layer="95" rot="R270"/>
+</segment>
+<segment>
+<pinref part="J5" gate="G$1" pin="1"/>
+<pinref part="SUPPLY2" gate="G$1" pin="GND2"/>
+<wire x1="157.48" y1="25.4" x2="152.4" y2="25.4" width="0.1524" layer="91"/>
+<label x="147.32" y="27.94" size="1.778" layer="95" rot="R270"/>
+</segment>
+<segment>
+<wire x1="109.22" y1="86.36" x2="109.22" y2="83.82" width="0.1524" layer="91"/>
+<label x="109.22" y="83.82" size="1.778" layer="95" rot="R180"/>
+<pinref part="U$2" gate="G$2" pin="P"/>
+</segment>
+</net>
+<net name="N$3" class="1">
+<segment>
+<wire x1="73.66" y1="81.28" x2="73.66" y2="78.74" width="0.1524" layer="91"/>
+<wire x1="73.66" y1="78.74" x2="73.66" y2="76.2" width="0.1524" layer="91"/>
+<wire x1="83.82" y1="81.28" x2="83.82" y2="78.74" width="0.1524" layer="91"/>
+<wire x1="83.82" y1="78.74" x2="73.66" y2="78.74" width="0.1524" layer="91"/>
+<junction x="73.66" y="78.74"/>
+<pinref part="Q1" gate="1" pin="D"/>
+<pinref part="U$1" gate="G$1" pin="2"/>
+<pinref part="U$2" gate="G$1" pin="2"/>
+</segment>
+</net>
+<net name="+12V" class="2">
 <segment>
 <wire x1="73.66" y1="91.44" x2="73.66" y2="99.06" width="0.1524" layer="91"/>
@@
 </segment>
 </net>
-<net name="!EMS" class="2">
-<segment>
-<pinref part="R2" gate="G$1" pin="1"/>
-<wire x1="45.72" y1="68.58" x2="33.02" y2="68.58" width="0.1524" layer="91"/>
-<label x="38.1" y="68.58" size="1.778" layer="95"/>
-</segment>
-</net>
-<net name="GND1" class="2">
-<segment>
-<pinref part="J7" gate="G$1" pin="2"/>
-<pinref part="SUPPLY7" gate="G$1" pin="GND2"/>
-<wire x1="27.94" y1="88.9" x2="33.02" y2="88.9" width="0.1524" layer="91"/>
-<label x="33.02" y="88.9" size="1.778" layer="95"/>
-</segment>
-<segment>
-<label x="99.06" y="116.84" size="1.778" layer="95"/>
-<wire x1="99.06" y1="96.52" x2="99.06" y2="101.6" width="0.1524" layer="91"/>
-<wire x1="99.06" y1="101.6" x2="99.06" y2="114.3" width="0.1524" layer="91"/>
-<wire x1="109.22" y1="96.52" x2="109.22" y2="101.6" width="0.1524" layer="91"/>
-<wire x1="109.22" y1="101.6" x2="99.06" y2="101.6" width="0.1524" layer="91"/>
-<junction x="99.06" y="101.6"/>
-<pinref part="U$1" gate="G$2" pin="O"/>
-<pinref part="U$2" gate="G$2" pin="O"/>
-</segment>
+<net name="GNDIO" class="2">
 <segment>
 <wire x1="73.66" y1="53.34" x2="73.66" y2="66.04" width="0.1524" layer="91"/>
@@
 </segment>
 </net>
-<net name="GND3" class="2">
-<segment>
-<pinref part="J4" gate="G$1" pin="1"/>
-<pinref part="SUPPLY3" gate="G$1" pin="GND2"/>
-<wire x1="157.48" y1="40.64" x2="152.4" y2="40.64" width="0.1524" layer="91"/>
-<label x="147.32" y="43.18" size="1.778" layer="95" rot="R270"/>
-</segment>
-<segment>
-<pinref part="J5" gate="G$1" pin="1"/>
-<pinref part="SUPPLY2" gate="G$1" pin="GND2"/>
-<wire x1="157.48" y1="25.4" x2="152.4" y2="25.4" width="0.1524" layer="91"/>
-<label x="147.32" y="27.94" size="1.778" layer="95" rot="R270"/>
-</segment>
-<segment>
-<wire x1="109.22" y1="86.36" x2="109.22" y2="83.82" width="0.1524" layer="91"/>
-<label x="109.22" y="83.82" size="1.778" layer="95" rot="R180"/>
-<pinref part="U$2" gate="G$2" pin="P"/>
-</segment>
-</net>
-<net name="N$3" class="1">
-<segment>
-<wire x1="73.66" y1="81.28" x2="73.66" y2="78.74" width="0.1524" layer="91"/>
-<wire x1="73.66" y1="78.74" x2="73.66" y2="76.2" width="0.1524" layer="91"/>
-<wire x1="83.82" y1="81.28" x2="83.82" y2="78.74" width="0.1524" layer="91"/>
-<wire x1="83.82" y1="78.74" x2="73.66" y2="78.74" width="0.1524" layer="91"/>
-<junction x="73.66" y="78.74"/>
-<pinref part="Q1" gate="1" pin="D"/>
-<pinref part="U$1" gate="G$1" pin="2"/>
-<pinref part="U$2" gate="G$1" pin="2"/>
-</segment>
-</net>
 </nets>
 </sheet>
@@
 <attribute name="VALUE" x="-10.16" y="22.86" size="1.778" layer="96" rot="R270"/>
 </instance>
-<instance part="F1" gate="G$1" x="-170.18" y="25.4" smashed="yes">
-<attribute name="NAME" x="-173.99" y="26.8986" size="1.778" layer="95"/>
-<attribute name="VALUE" x="-173.99" y="22.098" size="1.778" layer="96"/>
+<instance part="F1" gate="G$1" x="-137.16" y="25.4" smashed="yes">
+<attribute name="NAME" x="-140.97" y="26.8986" size="1.778" layer="95"/>
+<attribute name="VALUE" x="-140.97" y="22.098" size="1.778" layer="96"/>
 </instance>
 <instance part="GND23" gate="G$1" x="-7.62" y="15.24" smashed="yes" rot="R270">
@@
 <attribute name="VALUE" x="-13.97" y="-8.382" size="1.778" layer="96"/>
 </instance>
-<instance part="C1" gate="G$1" x="-147.32" y="22.86" smashed="yes">
-<attribute name="NAME" x="-145.796" y="23.241" size="1.778" layer="95"/>
-<attribute name="VALUE" x="-145.796" y="18.161" size="1.778" layer="96"/>
-</instance>
-<instance part="C2" gate="G$1" x="-137.16" y="22.86" smashed="yes">
-<attribute name="NAME" x="-136.017" y="23.3426" size="1.778" layer="95"/>
-<attribute name="VALUE" x="-136.017" y="18.2626" size="1.778" layer="96"/>
+<instance part="C1" gate="G$1" x="-127" y="22.86" smashed="yes">
+<attribute name="NAME" x="-125.476" y="23.241" size="1.778" layer="95"/>
+<attribute name="VALUE" x="-125.476" y="18.161" size="1.778" layer="96"/>
 </instance>
 <instance part="GND1" gate="G$1" x="-20.32" y="-5.08" smashed="yes" rot="R270">
@@
 <wire x1="-15.24" y1="-5.08" x2="-17.78" y2="-5.08" width="0.1524" layer="91"/>
 <pinref part="GND1" gate="G$1" pin="GNDIO"/>
+</segment>
+<segment>
+<pinref part="R30" gate="G$1" pin="1"/>
+<wire x1="-104.14" y1="2.54" x2="-104.14" y2="5.08" width="0.1524" layer="91"/>
+<label x="-104.14" y="2.54" size="1.778" layer="95"/>
+</segment>
+<segment>
+<pinref part="C1" gate="G$1" pin="2"/>
+<wire x1="-127" y1="17.78" x2="-127" y2="12.7" width="0.1524" layer="91"/>
+<label x="-127" y="12.7" size="1.778" layer="95"/>
 </segment>
 </net>
@@
 </segment>
 </net>
-<net name="BATT_POWER" class="2">
-<segment>
-<pinref part="F1" gate="G$1" pin="1"/>
-<wire x1="-195.58" y1="25.4" x2="-175.26" y2="25.4" width="0.1524" layer="91"/>
-<label x="-193.04" y="25.4" size="1.778" layer="95"/>
-</segment>
-</net>
 <net name="N$5" class="0">
 <segment>
@@
 <label x="-15.24" y="10.16" size="1.778" layer="95"/>
 </segment>
-</net>
-<net name="GND1" class="2">
-<segment>
-<pinref part="R30" gate="G$1" pin="1"/>
-<wire x1="-104.14" y1="2.54" x2="-104.14" y2="5.08" width="0.1524" layer="91"/>
-<label x="-104.14" y="2.54" size="1.778" layer="95"/>
-</segment>
-<segment>
-<pinref part="C1" gate="G$1" pin="2"/>
-<wire x1="-147.32" y1="17.78" x2="-147.32" y2="15.24" width="0.1524" layer="91"/>
-<pinref part="C2" gate="G$1" pin="-"/>
-<wire x1="-137.16" y1="17.78" x2="-137.16" y2="15.24" width="0.1524" layer="91"/>
-<wire x1="-137.16" y1="15.24" x2="-147.32" y2="15.24" width="0.1524" layer="91"/>
-<wire x1="-147.32" y1="15.24" x2="-147.32" y2="12.7" width="0.1524" layer="91"/>
-<junction x="-147.32" y="15.24"/>
-<label x="-147.32" y="12.7" size="1.778" layer="95"/>
+<segment>
+<pinref part="F1" gate="G$1" pin="1"/>
+<wire x1="-147.32" y1="25.4" x2="-142.24" y2="25.4" width="0.1524" layer="91"/>
+<label x="-147.32" y="25.4" size="1.778" layer="95"/>
 </segment>
 </net>
@@
 <pinref part="U4" gate="G$1" pin="C"/>
 <label x="-104.14" y="25.4" size="1.778" layer="95"/>
-<wire x1="-165.1" y1="25.4" x2="-147.32" y2="25.4" width="0.1524" layer="91"/>
+<wire x1="-132.08" y1="25.4" x2="-127" y2="25.4" width="0.1524" layer="91"/>
 <pinref part="C1" gate="G$1" pin="1"/>
-<pinref part="C2" gate="G$1" pin="+"/>
-<wire x1="-137.16" y1="25.4" x2="-147.32" y2="25.4" width="0.1524" layer="91"/>
-<wire x1="-137.16" y1="25.4" x2="-99.06" y2="25.4" width="0.1524" layer="91"/>
+<wire x1="-127" y1="25.4" x2="-99.06" y2="25.4" width="0.1524" layer="91"/>
 <pinref part="F1" gate="G$1" pin="2"/>
-<junction x="-147.32" y="25.4"/>
-<junction x="-137.16" y="25.4"/>
-</segment>
-</net>
+<junction x="-127" y="25.4"/>
+</segment>
+</net>
